File: 2812-32/2812-32-mini/2812-32-mini.kicad_pcb (KiCad board)
At the start: 2 copper layers, 26.2 x 54.1 mm, 42 parts, among them J1 USB-C, J2 I2C_STANDARDQWIIC, SW1 SW_DIP_x01, U2 ESP32-C3-MINI-1, U3 LM2575-3.3BU, U4 HUSB238

Commit message: mini
Parts:
- removed FET2: AONR21307, Package_DFN_QFN:DFN-10-1EP_3x3mm_P0.5mm_EP1.58x2.35mm
- added Q1: SI7611DN-T1-GE3, S176etc:MOSFET_0DN-T1-GE3_VIS, F.Cu at (90.3, 60.1)
Connections:
- U3 pad 4: unconnected-(U3-FB-Pad4) -> +3.3V
Routing:
- net +3.3V: track 116.9 -> 127.1 mm, vias 5 -> 7
- net Net-(U4-VIN): track 13.8 -> 19.5 mm
- net Net-(Q1-G): track 13.7 -> 10.6 mm
- net GPIO10: track 27.7 -> 26.4 mm, vias 1 -> 0
- net VDC: track 39.7 -> 40.6 mm
