File: 2812-32/2812-32-mini/CONN.kicad_sch (KiCad schematic)
At the start: 4 parts, among them J10 I2C_STANDARDQWIIC

Commit message: mini
Parts:
- CH2, CHO1: MPN (none) -> C265360
- J10: MPN (none) -> C160404
