File: 2812-32/2812-32-mini/Power.kicad_sch (KiCad schematic)
At the start: 11 parts, among them U3 LM2575-3.3BU

Commit message: mini
Parts:
- C6: MPN (none) -> C5354996
- C7: MPN (none) -> C2980164
- D1: MPN (none) -> C437199
- D2, D3, D4: MPN (none) -> C5656657
- L1: MPN (none) -> C394139
- R7, R8, R9: MPN (none) -> C2906961
- U3: MPN (none) -> C2977107
Connections:
- net +3.3V: now also U3.4 (FB)
