File: 2812-32/2812-32-mini/esp32.kicad_sch (KiCad schematic)
At the start: 9 parts, among them SW1 SW_DIP_x01, U2 ESP32-C3-MINI-1

Commit message: mini
Parts:
- C31: MPN (none) -> C15525
- C32: MPN (none) -> C20539426
- C33, C9: MPN (none) -> C307331
- R10, R11, R31: MPN (none) -> C25744
- SW1: MPN (none) -> C231329
- U2: MPN (none) -> C2838502
