File: 2812-32/2812-32-mini/usb.kicad_sch (KiCad schematic)
At the start: 15 parts, among them J1 USB-C, U4 HUSB238

Commit message: mini
Parts:
- removed FET2: AONR21307, Package_DFN_QFN:DFN-10-1EP_3x3mm_P0.5mm_EP1.58x2.35mm, symbol AONR21307:AONR21307
- added Q1: SI7611DN-T1-GE3, MOSFET_0DN-T1-GE3_VIS, symbol SI7611DN-T1-GE3:SI7619DN-T1-GE3
- 5v    12v1: MPN (none) -> C20607074
- C35, C36: MPN (none) -> C1671
- C8: MPN (none) -> C20539426
- J1: MPN (none) -> C2988369
- R34, R36: MPN (none) -> C2930077
- R4, RR1, RR2: MPN (none) -> C25905
- R5: MPN (none) -> C409918
- R6: MPN (none) -> C25744
- RS1: MPN (none) -> C4216
- U4: MPN (none) -> C7471904
Connections:
- net VDC: now also Q1.5 (D), Q1.6 (D), Q1.7 (D), Q1.8 (D)
- net at C8.1, J1.A4 (VBUS), J1.A9 (VBUS)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: now also Q1.1 (S), Q1.2 (S), Q1.3 (S)
- net at R4.1, R5.1: now also Q1.4 (G)
Other:
- moved on the sheet: 5v 12v1, C35, C36, C8, J1, R34, R36, R4, R5, R6, RR1, RR2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
